File: Battery Shield/battery-shield-smallinductor/EAGLE/Battery Shield.brd (EAGLE design)
At the start: 58.5 x 15.2 mm, 32 parts, among them IC1 MCP73871, U1 TPS61200

Commit message: added license info to all design files
Other:
- board text added: "Reference Designs ARE PROVIDED "AS IS" AND "WITH ALL FAULTS. SPARK LABS, INC ("SPARK") DISCLAIMS ALL OTHER WARRANTIES, EXPRESS OR IMPLIED, REGARDING PRODUCTS OR THE REFERENCE DESIGNS, INCLUDING BUT NOT LIMITED TO, ANY IMPLIED WARRANTIES OF MERCHANTABILITY, FITNESS FOR A PARTICULAR PURPOSE, OR NON-INFRINGEMENT. Spark may make changes to specifications and product descriptions at any time, without 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"
Changed lines of the file:
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@@
 <layer number="49" name="Reference" color="7" fill="1" visible="no" active="yes"/>
 <layer number="50" name="dxf" color="7" fill="1" visible="no" active="no"/>
-<layer number="51" name="tDocu" color="6" fill="1" visible="no" active="yes"/>
+<layer number="51" name="tDocu" color="6" fill="1" visible="yes" active="yes"/>
 <layer number="52" name="bDocu" color="7" fill="1" visible="no" active="yes"/>
 <layer number="53" name="tGND_GNDA" color="7" fill="9" visible="no" active="no"/>
@@
 <wire x1="72.009" y1="2.159" x2="69.215" y2="0.762" width="0.0254" layer="20" curve="-13.69593"/>
 <text x="36.2712" y="0.4318" size="1.778" layer="22" rot="MR0">+</text>
+<text x="96.52" y="2.54" size="1.27" layer="51">Reference Designs ARE PROVIDED "AS IS" AND "WITH ALL FAULTS. SPARK LABS, INC
+("SPARK") DISCLAIMS ALL OTHER WARRANTIES, EXPRESS OR IMPLIED, REGARDING
+PRODUCTS OR THE REFERENCE DESIGNS, INCLUDING BUT NOT LIMITED TO, ANY
+IMPLIED WARRANTIES OF MERCHANTABILITY, FITNESS FOR A PARTICULAR PURPOSE,
+OR NON-INFRINGEMENT.
+Spark may make changes to specifications and product descriptions at any
+time, without notice. The Customer must not rely on the absence or
+characteristics of any features or instructions marked "reserved" or
+"undefined." Spark reserves these for future definition and shall have
+no responsibility whatsoever for conflicts or incompatibilities arising
+from future changes to them. The product information on the Web Site or
+Materials is subject to change without notice. Do not finalize a design
+with this information.
+Spark is a registered trademark.</text>
+<wire x1="93.98" y1="0" x2="93.98" y2="33.02" width="0.4064" layer="51"/>
+<wire x1="93.98" y1="33.02" x2="177.8" y2="33.02" width="0.4064" layer="51"/>
+<wire x1="177.8" y1="33.02" x2="177.8" y2="0" width="0.4064" layer="51"/>
+<wire x1="177.8" y1="0" x2="93.98" y2="0" width="0.4064" layer="51"/>
 </plain>
 <attributes>

Commit message: updated battery shield gerbers to v201
Parts:
- removed C2: 0.1uF, SparkFun-Passives:0402-CAP
- added R14: 10K, SparkFun-Passives:0402-RES
- added SJ2: SOLDERJUMPERNO, SparkFun-Passives:SJ_2S-NO
- moved LED1 7.44 mm to (25.0, 5.71)
- moved LED3 7.44 mm to (66.9, 5.71)
- moved R6 2.77 mm to (53.6, 2.08)
- moved R11 2.67 mm to (49.4, 7.24)
- moved R12 2.29 mm to (49.7, 4.06)
- moved R13 2.29 mm to (50.9, 4.06)
- moved RT1 2.29 mm to (52.2, 4.06)
- moved RT2 2.29 mm to (53.5, 4.06), turned to 90 degrees
- moved U$2 1.44 mm to (67.3, 5.23)
- moved C3 1.20 mm to (24.5, 5.21)
- moved R3 0.89 mm to (35.3, 11.7)
- moved R10 0.77 mm to (57.0, 4.06)
- moved JP1 0.38 mm to (61.7, 1.91)
Connections:
- new net N$20: IC1.3, R14.2, SJ2.2
- net GND: now also R14.1
- net N$3: no longer C2.2
- net VBATT_OUT: no longer C2.1
- net VBUS: now also SJ2.1; no longer IC1.3
Routing:
- net VBUS: track 104.4 -> 90.4 mm, vias 5 -> 6
- net N$8: track 37.4 -> 28.2 mm
- net N$20: track 0.00 -> 7.62 mm
- net N$16: track 24.7 -> 17.9 mm
- net GND: track 45.3 -> 51.4 mm
- net N$10: track 7.10 -> 3.72 mm
- net N$6: track 5.18 -> 3.32 mm
- net N$12: track 7.30 -> 8.35 mm
- net N$14: track 4.85 -> 5.75 mm
- net VBATT_OUT: track 40.1 -> 40.7 mm
- net N$9: track 3.87 -> 3.36 mm
Other:
- board size 58.5 x 15.2 mm -> 48.3 x 15.4 mm
- board text added: "Battery Shield v2.0.1"
- board text added: "J1"
- board text added: "J2"
- board text added: "spark.io"
- board text removed: "Battery Shield"
