File: electron-shields/asset-tracker/eagle/asset-tracker-v003/asset-tracker-v003.brd (EAGLE design)
At the start: 95.2 x 38.1 mm, 23 parts, among them J1 1X2-3.5MM, T1 DMG3415, U1 FGPMMOPA6H, U3 LIS3DHTR, X1 ELECTRON, X2 uFL

Commit message: v002 updates and creation of future v003
Parts:
- removed JP4: (no value), microbuilder:1X01_ROUND
- added C6: 1uF, microbuilder:0805-NO@1
- added X3: BU-SMA-V, con-coax:BU-SMA-V
- C1: value 0.1uF -> 0.01uF
- R7: value 10K -> 2K2
- moved U$13 38.5 mm to (33.5, 40.0)
- moved U$21 37.8 mm to (21.2, 39.5)
- moved X2 35.7 mm to (-7.62, 4.32)
- moved J1 30.7 mm to (25.1, 34.4), turned to 180 degrees
- moved B1 24.1 mm to (10.5, 31.5), turned to 0 degrees
- moved U1 20.5 mm to (19.8, 9.02), turned to 270 degrees
- moved D1 19.1 mm to (25.3, 28.8)
- moved JP2 19.0 mm to (7.75, 11.9)
- moved LED1 15.3 mm to (1.52, 13.2), turned to 180 degrees
- moved R1 13.1 mm to (3.43, 13.2), turned to 270 degrees
- moved C2 11.8 mm to (28.4, 24.5), turned to 270 degrees
- moved R7 9.53 mm to (23.0, 24.6), turned to 270 degrees
- moved R8 9.29 mm to (19.4, 27.4), turned to 90 degrees
- moved T1 9.27 mm to (25.7, 24.6), turned to 90 degrees
- moved C1 5.02 mm to (23.9, 20.6), turned to 90 degrees
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Connections:
- net D6: no longer JP4.1
- net GND: now also C6.2, J1.2, X3.2, X3.3, X3.4, X3.5; no longer J1.1, X2.1, X2.2
- net N$4: now also X3.1; no longer X2.3
- net N$9: now also J1.1; no longer J1.2
- net VBACKUP: now also C6.1
Routing:
- net D6: track 97.3 -> 42.5 mm
- net ACCEL_CS: track 67.0 -> 104.0 mm
- net 3.3V: track 80.1 -> 43.9 mm, vias 7 -> 6
- net ACCEL_MISO: track 57.7 -> 85.8 mm, vias 2 -> 1
- net ACCEL_INT1: track 52.2 -> 79.8 mm, vias 2 -> 1
- net ACCEL_MOSI: track 57.3 -> 84.2 mm, vias 2 -> 1
- net GND: track 69.4 -> 54.0 mm, vias 6 -> 25
- net TX: track 61.4 -> 73.4 mm
- net 1PPS: track 5.51 -> 16.8 mm, vias 0 -> 1
- net RX: track 56.8 -> 65.5 mm, vias 1 -> 0
- net ACCEL_SCK: track 82.6 -> 90.4 mm
- net N$4: track 3.06 -> 10.7 mm
- net N$1: track 6.94 -> 13.1 mm
- net N$8: track 44.5 -> 40.4 mm
- net VBACKUP: track 28.5 -> 32.3 mm, vias 2 -> 0
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- added copper zone on layer 16, net GND
Other:
- outline, holes or cut-outs redrawn
- board text removed: "VIN = 5V to 12VDC"
