File: electron-shields/asset-tracker/eagle/asset-tracker-v003/asset-tracker-v003.sch (EAGLE design)
At the start: 21 parts, among them J1 1X2-3.5MM, T1 DMG3415, U1 FGPMMOPA6H, U3 LIS3DHTR, X1 ELECTRON, X2 uFL

Commit message: v002 updates and creation of future v003
Parts:
- removed JP4: (no value), microbuilder:HEADER-1X1ROUND
- added C6: 1uF, microbuilder:CAP_CERAMIC0805-NOOUTLINE
- added X3: BU-SMA-V, con-coax:BU-SMA-V
- C1: value 0.1uF -> 0.01uF
- R7: value 10K -> 2K2
Connections:
- net D6: no longer JP4.1
- net GND: now also C6.2, J1.2, X3.2; no longer J1.1, X2.GND@0, X2.GND@1
- net N$4: now also X3.1; no longer X2.SIGNAL
- net N$9: now also J1.1; no longer J1.2
- net VBACKUP: now also C6.1
Changed lines of the file:
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@@
 <setting verticaltext="up"/>
 </settings>
-<grid distance="0.1" unitdist="inch" unit="inch" style="lines" multiple="1" display="no" altdistance="0.01" altunitdist="inch" altunit="inch"/>
+<grid distance="0.05" unitdist="inch" unit="inch" style="lines" multiple="1" display="yes" altdistance="0.01" altunitdist="inch" altunit="inch"/>
 <layers>
 <layer number="1" name="Top" color="4" fill="1" visible="no" active="no"/>
@@
 <layer number="112" name="tSilk" color="7" fill="1" visible="yes" active="yes"/>
 <layer number="113" name="LOGO" color="7" fill="1" visible="yes" active="yes"/>
+<layer number="114" name="Badge_Outline" color="7" fill="1" visible="no" active="yes"/>
+<layer number="115" name="ReferenceISLANDS" color="7" fill="1" visible="no" active="yes"/>
 <layer number="116" name="Patch_BOT" color="9" fill="4" visible="yes" active="yes"/>
 <layer number="118" name="Rect_Pads" color="7" fill="1" visible="yes" active="yes"/>
@@
 <part name="R1" library="microbuilder" deviceset="RESISTOR" device="0805_NOOUTLINE" value="470-1K"/>
 <part name="U$2" library="microbuilder" deviceset="GND" device=""/>
-<part name="C1" library="microbuilder" deviceset="CAP_CERAMIC" device="0805-NOOUTLINE" value="0.1uF"/>
+<part name="C1" library="microbuilder" deviceset="CAP_CERAMIC" device="0805-NOOUTLINE" value="0.01uF"/>
 <part name="B1" library="microbuilder" deviceset="BATTERY" device="CR1220_SMT" value="CR1220"/>
 <part name="U$14" library="microbuilder" deviceset="GND" device=""/>
@@
 <part name="JP3" library="microbuilder" deviceset="HEADER-1X15" device=""/>
 <part name="T1" library="zetex" deviceset="PMOSSOT23" device="" value="DMG3415"/>
-<part name="R7" library="microbuilder" deviceset="RESISTOR" device="0805_NOOUTLINE" value="10K"/>
+<part name="R7" library="microbuilder" deviceset="RESISTOR" device="0805_NOOUTLINE" value="2K2"/>
 <part name="U$15" library="microbuilder" deviceset="3.3V" device=""/>
-<part name="JP4" library="microbuilder" deviceset="HEADER-1X1" device="ROUND"/>
+<part name="C6" library="microbuilder" deviceset="CAP_CERAMIC" device="0805-NOOUTLINE" value="1uF"/>
+<part name="X3" library="con-coax" deviceset="BU-SMA-V" device=""/>
+<part name="U$4" library="microbuilder" deviceset="GND" device=""/>
 </parts>
 <sheets>
@@
 <instance part="C2" gate="G$1" x="48.26" y="162.56" rot="R90"/>
 <instance part="U$5" gate="G$1" x="50.8" y="160.02"/>
-<instance part="J1" gate="G$1" x="43.18" y="180.34" rot="R90"/>
+<instance part="J1" gate="G$1" x="40.64" y="179.07" rot="MR90"/>
 <instance part="U$1" gate="G$1" x="109.22" y="144.78" rot="R90"/>
 <instance part="D1" gate="G$1" x="43.18" y="170.18" rot="R270"/>
@@
 <instance part="R7" gate="G$1" x="180.34" y="167.64" rot="R90"/>
 <instance part="U$15" gate="G$1" x="172.72" y="180.34"/>
-<instance part="JP4" gate="G$1" x="200.66" y="165.1" rot="R90"/>
+<instance part="C6" gate="G$1" x="232.41" y="153.67"/>
+<instance part="X3" gate="G$1" x="231.14" y="101.6" rot="MR0"/>
+<instance part="U$4" gate="G$1" x="228.6" y="91.44"/>
 </instances>
 <busses>
@@
 <segment>
 <wire x1="218.44" y1="119.38" x2="238.76" y2="119.38" width="0.1524" layer="91"/>
-<wire x1="238.76" y1="119.38" x2="238.76" y2="111.76" width="0.1524" layer="91"/>
-<wire x1="238.76" y1="111.76" x2="238.76" y2="109.22" width="0.1524" layer="91"/>
-<wire x1="238.76" y1="109.22" x2="238.76" y2="106.68" width="0.1524" layer="91"/>
+<wire x1="238.76" y1="119.38" x2="238.76" y2="106.68" width="0.1524" layer="91"/>
 <wire x1="218.44" y1="137.16" x2="238.76" y2="137.16" width="0.1524" layer="91"/>
 <wire x1="238.76" y1="137.16" x2="238.76" y2="119.38" width="0.1524" layer="91"/>
-<wire x1="231.14" y1="109.22" x2="238.76" y2="109.22" width="0.1524" layer="91"/>
-<wire x1="231.14" y1="111.76" x2="238.76" y2="111.76" width="0.1524" layer="91"/>
 <junction x="238.76" y="119.38"/>
-<junction x="238.76" y="109.22"/>
-<junction x="238.76" y="111.76"/>
 <pinref part="U1" gate="G$1" pin="GND@3"/>
 <pinref part="U$19" gate="G$1" pin="GND"/>
 <pinref part="U1" gate="G$1" pin="GND@4"/>
-<pinref part="X2" gate="G$1" pin="GND@1"/>
-<pinref part="X2" gate="G$1" pin="GND@0"/>
-</segment>
-<segment>
-<wire x1="241.3" y1="152.4" x2="241.3" y2="147.32" width="0.1524" layer="91"/>
+</segment>
+<segment>
+<wire x1="241.3" y1="152.4" x2="241.3" y2="149.86" width="0.1524" layer="91"/>
 <pinref part="B1" gate="G$1" pin="-"/>
 <pinref part="U$14" gate="G$1" pin="GND"/>
+<pinref part="C6" gate="G$1" pin="2"/>
+<wire x1="241.3" y1="149.86" x2="241.3" y2="147.32" width="0.1524" layer="91"/>
+<wire x1="232.41" y1="151.13" x2="232.41" y2="149.86" width="0.1524" layer="91"/>
+<wire x1="232.41" y1="149.86" x2="241.3" y2="149.86" width="0.1524" layer="91"/>
+<junction x="241.3" y="149.86"/>
 </segment>
 <segment>
@@
 </segment>
 <segment>
-<pinref part="U$3" gate="G$1" pin="GND"/>
-<wire x1="40.64" y1="175.26" x2="40.64" y2="157.48" width="0.1524" layer="91"/>
-<pinref part="J1" gate="G$1" pin="1"/>
-</segment>
-<segment>
 <pinref part="C2" gate="G$1" pin="2"/>
 <pinref part="U$5" gate="G$1" pin="GND"/>
@@
 <pinref part="JP1" gate="G$1" pin="4"/>
 </segment>
+<segment>
+<pinref part="X3" gate="G$1" pin="2"/>
+<wire x1="228.6" y1="99.06" x2="228.6" y2="93.98" width="0.1524" layer="91"/>
+<pinref part="U$4" gate="G$1" pin="GND"/>
+</segment>
+<segment>
+<pinref part="U$3" gate="G$1" pin="GND"/>
+<pinref part="J1" gate="G$1" pin="2"/>
+<wire x1="40.64" y1="157.48" x2="40.64" y2="173.99" width="0.1524" layer="91"/>
+</segment>
 </net>
 <net name="3.3V" class="0">
@@
 </segment>
 <segment>
-<wire x1="241.3" y1="157.48" x2="241.3" y2="167.64" width="0.1524" layer="91"/>
+<wire x1="241.3" y1="157.48" x2="241.3" y2="160.02" width="0.1524" layer="91"/>
 <label x="241.3" y="160.02" size="1.778" layer="95" rot="R90"/>
 <pinref part="B1" gate="G$1" pin="+"/>
+<pinref part="C6" gate="G$1" pin="1"/>
+<wire x1="241.3" y1="160.02" x2="241.3" y2="167.64" width="0.1524" layer="91"/>
+<wire x1="232.41" y1="158.75" x2="232.41" y2="160.02" width="0.1524" layer="91"/>
+<wire x1="232.41" y1="160.02" x2="241.3" y2="160.02" width="0.1524" layer="91"/>
+<junction x="241.3" y="160.02"/>
 </segment>
 </net>
@@
 <junction x="55.88" y="147.32"/>
 <pinref part="JP3" gate="G$1" pin="13"/>
-</segment>
-</net>
-<net name="N$4" class="0">
-<segment>
-<wire x1="218.44" y1="116.84" x2="223.52" y2="116.84" width="0.1524" layer="91"/>
-<pinref part="U1" gate="G$1" pin="EX_ANT"/>
-<pinref part="X2" gate="G$1" pin="SIGNAL"/>
 </segment>
 </net>
@@
 <segment>
 <wire x1="180.34" y1="162.56" x2="177.8" y2="162.56" width="0.1524" layer="91"/>
-<junction x="180.34" y="162.56"/>
 <pinref part="R7" gate="G$1" pin="1"/>
 <pinref part="T1" gate="A" pin="G"/>
-<wire x1="180.34" y1="162.56" x2="200.66" y2="162.56" width="0.1524" layer="91"/>
-<label x="193.04" y="162.56" size="1.778" layer="95"/>
-<pinref part="JP4" gate="G$1" pin="1"/>
+<label x="177.8" y="160.02" size="1.778" layer="95"/>
 </segment>
 </net>
@@
 </segment>
 </net>
-<net name="N$9" class="0">
-<segment>
-<pinref part="D1" gate="G$1" pin="A"/>
-<pinref part="J1" gate="G$1" pin="2"/>
-<wire x1="43.18" y1="172.72" x2="43.18" y2="175.26" width="0.1524" layer="91"/>
-</segment>
-</net>
 <net name="VCC" class="0">
 <segment>
@@
 </segment>
 </net>
+<net name="N$4" class="0">
+<segment>
+<pinref part="U1" gate="G$1" pin="EX_ANT"/>
+<wire x1="218.44" y1="116.84" x2="220.98" y2="116.84" width="0.1524" layer="91"/>
+<wire x1="220.98" y1="116.84" x2="220.98" y2="101.6" width="0.1524" layer="91"/>
+<pinref part="X3" gate="G$1" pin="1"/>
+<wire x1="220.98" y1="101.6" x2="228.6" y2="101.6" width="0.1524" layer="91"/>
+</segment>
+</net>
+<net name="N$9" class="0">
+<segment>
+<pinref part="D1" gate="G$1" pin="A"/>
+<pinref part="J1" gate="G$1" pin="1"/>
+<wire x1="43.18" y1="173.99" x2="43.18" y2="172.72" width="0.1524" layer="91"/>
+</segment>
+</net>
