File: electron-shields/asset-tracker/eagle/asset-tracker-v004/asset-tracker-v004.brd (EAGLE design)
At the start: 103 x 36 mm, 30 parts, among them J1 1X2-3.5MM, T1 DMG3415, U1 MAX-M8, U2 MAX2674, U3 LIS3DHTR, U4 EPCOS-B9444, U5 MS621FE, X1 ELECTRON, X2 IPEX-20279-001E

Commit message: added a nuclear reactor for power, routing done, need labels
Parts:
- removed R2: 100K, rcl:R0402
- moved C4 0.51 mm to (65.0, 3.56)
- moved C10 0.40 mm to (69.9, 15.7)
- moved C5 0.30 mm to (66.4, 17.4)
- moved C6 0.30 mm to (73.0, 17.8)
- moved L1 0.30 mm to (70.9, 17.8)
- moved U2 0.30 mm to (69.1, 17.7)
Connections:
- net GND: now also A1.1, A1.2, A1.3, A1.4
- net GPS_!RESET: no longer R2.1
- net GPS_VCC: no longer R2.2
- net N$12: now also A1.0; no longer A1.ANT
Routing:
- net 3.3V: track 95.5 -> 24.7 mm
- net N$11: track 0.00 -> 61.0 mm
- net N$53: track 0.00 -> 10.7 mm
- net N$31: track 0.00 -> 10.4 mm, vias 0 -> 1
- net N$30: track 0.00 -> 10.4 mm, vias 0 -> 1
- net N$28: track 0.00 -> 10.4 mm, vias 0 -> 1
- net N$26: track 0.00 -> 10.4 mm, vias 0 -> 1
- net N$25: track 0.00 -> 10.4 mm, vias 0 -> 1
- net N$23: track 0.00 -> 10.4 mm, vias 0 -> 1
- net N$20: track 0.00 -> 10.4 mm, vias 0 -> 1
- net N$19: track 0.00 -> 10.4 mm, vias 0 -> 1
- net N$18: track 0.00 -> 10.4 mm, vias 0 -> 1
- net N$17: track 0.00 -> 10.4 mm, vias 0 -> 1
- net N$14: track 0.00 -> 10.4 mm, vias 0 -> 1
- net N$13: track 0.00 -> 10.4 mm, vias 0 -> 1
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- added copper zone on layer 15, net 3.3V
- added copper zone on layer 2, net GND
