File: electron-shields/asset-tracker/eagle/asset-tracker-v004/asset-tracker-v004.brd (EAGLE design)
At the start: 103 x 36 mm, 29 parts, among them J1 1X2-3.5MM, T1 DMG3415, U1 MAX-M8, U2 MAX2674, U3 LIS3DHTR, U4 EPCOS-B9444, U5 MS621FE, X1 ELECTRON, X2 IPEX-20279-001E

Commit message: added labels in gotham font, needs aligning
Parts:
- added JP3, JP4, JP5, JP6, JP7: (no value), SparkFun-Connectors:1X01NS-KIT
- moved C2 3.90 mm to (57.0, 23.2), turned to 270 degrees
- moved R8 2.16 mm to (32.0, 20.5)
Connections:
- net GPS_!RESET: now also JP6.1
- net GPS_!SAFEBOOT: now also JP5.1
- net GPS_EXTINT: now also JP7.1
- net GPS_SCL: now also JP3.1
- net GPS_SDA: now also JP4.1
Routing:
- net GPS_!RESET: track 0.00 -> 23.8 mm, vias 0 -> 1
- net GPS_EXTINT: track 0.00 -> 19.7 mm, vias 0 -> 1
- net N$53: track 10.7 -> 0.00 mm
- net N$31: track 10.4 -> 0.00 mm, vias 1 -> 0
- net N$30: track 10.4 -> 0.00 mm, vias 1 -> 0
- net N$28: track 10.4 -> 0.00 mm, vias 1 -> 0
- net N$26: track 10.4 -> 0.00 mm, vias 1 -> 0
- net N$25: track 10.4 -> 0.00 mm, vias 1 -> 0
- net N$23: track 10.4 -> 0.00 mm, vias 1 -> 0
- net N$20: track 10.4 -> 0.00 mm, vias 1 -> 0
- net N$19: track 10.4 -> 0.00 mm, vias 1 -> 0
- net N$18: track 10.4 -> 0.00 mm, vias 1 -> 0
- net N$17: track 10.4 -> 0.00 mm, vias 1 -> 0
- net N$14: track 10.4 -> 0.00 mm, vias 1 -> 0
- net N$13: track 10.4 -> 0.00 mm, vias 1 -> 0
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Other:
- board text added: "/Users/mohitbhoite/particle/shields/electron-shields/asset-tracker/eagle/asset-tracker-v004/LABELS.BMP"

Commit message: labeling done
Parts:
- removed U5: MS621FE, Explore Labs EAGLE Library:MS621FE
- added C1: (no value), adafruit:414-VA5R
- moved R5 0.75 mm to (49.4, 18.0)
- moved D3 0.73 mm to (52.5, 18.0)
Connections:
- net GND: now also C1.-; no longer U5.NEG
- net N$7: now also C1.+; no longer U5.POS
Routing:
- net GPS_PWR_EN: track 34.4 -> 30.8 mm
- net N$24: track 0.00 -> 1.78 mm
- net N$23: track 0.00 -> 1.78 mm
- net N$13: track 0.00 -> 1.78 mm
- net N$22: track 0.00 -> 1.52 mm
- net N$21: track 0.00 -> 1.52 mm
- net N$20: track 0.00 -> 1.52 mm
- net N$19: track 0.00 -> 1.52 mm
- net N$18: track 0.00 -> 1.52 mm
- net N$17: track 0.00 -> 1.52 mm
- net N$14: track 0.00 -> 1.52 mm
- net N$36: track 0.00 -> 1.52 mm
- net N$35: track 0.00 -> 1.52 mm
- net N$34: track 0.00 -> 1.52 mm
- net N$33: track 0.00 -> 1.52 mm
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Other:
- board text removed: "/Users/mohitbhoite/particle/shields/electron-shields/asset-tracker/eagle/asset-tracker-v004/LABELS.BMP"
