File: electron-shields/asset-tracker/eagle/asset-tracker-v004/asset-tracker-v004.sch (EAGLE design)
At the start: 29 parts, among them J1 1X2-3.5MM, T1 DMG3415, U1 MAX-M8, U2 MAX2674, U3 LIS3DHTR, U4 EPCOS-B9444, U5 MS621FE, X1 ELECTRON, X2 IPEX-20279-001E

Commit message: added labels in gotham font, needs aligning
Parts:
- added JP3, JP4, JP5, JP6, JP7: (no value), SparkFun-Connectors:M01NOSILK-KIT
Connections:
- net GPS_!RESET: now also JP6.1
- net GPS_!SAFEBOOT: now also JP5.1
- net GPS_EXTINT: now also JP7.1
- net GPS_SCL: now also JP3.1
- net GPS_SDA: now also JP4.1
Changed lines of the file:
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@@
 <part name="U5" library="Explore Labs EAGLE Library" deviceset="MS621FE" device=""/>
 <part name="U$28" library="microbuilder" deviceset="GND" device=""/>
+<part name="JP3" library="SparkFun-Connectors" deviceset="M01" device="NOSILK-KIT"/>
+<part name="JP4" library="SparkFun-Connectors" deviceset="M01" device="NOSILK-KIT"/>
+<part name="JP5" library="SparkFun-Connectors" deviceset="M01" device="NOSILK-KIT"/>
+<part name="JP6" library="SparkFun-Connectors" deviceset="M01" device="NOSILK-KIT"/>
+<part name="JP7" library="SparkFun-Connectors" deviceset="M01" device="NOSILK-KIT"/>
 </parts>
 <sheets>
@@
 <instance part="U5" gate="G$1" x="236.22" y="158.75" rot="R90"/>
 <instance part="U$28" gate="G$1" x="8.89" y="153.67"/>
+<instance part="JP3" gate="G$1" x="224.79" y="115.57" rot="R180"/>
+<instance part="JP4" gate="G$1" x="224.79" y="118.11" rot="R180"/>
+<instance part="JP5" gate="G$1" x="129.54" y="115.57"/>
+<instance part="JP6" gate="G$1" x="129.54" y="120.65"/>
+<instance part="JP7" gate="G$1" x="129.54" y="123.19"/>
 </instances>
 <busses>
@@
 <wire x1="201.93" y1="118.11" x2="217.17" y2="118.11" width="0.1524" layer="91"/>
 <label x="203.2" y="118.11" size="1.778" layer="95"/>
+<pinref part="JP4" gate="G$1" pin="1"/>
 </segment>
 </net>
@@
 <wire x1="201.93" y1="115.57" x2="217.17" y2="115.57" width="0.1524" layer="91"/>
 <label x="203.2" y="115.57" size="1.778" layer="95"/>
+<pinref part="JP3" gate="G$1" pin="1"/>
 </segment>
 </net>
@@
 <wire x1="158.75" y1="123.19" x2="137.16" y2="123.19" width="0.1524" layer="91"/>
 <label x="137.16" y="123.19" size="1.778" layer="95"/>
+<pinref part="JP7" gate="G$1" pin="1"/>
 </segment>
 </net>
@@
 <wire x1="158.75" y1="120.65" x2="137.16" y2="120.65" width="0.1524" layer="91"/>
 <label x="137.16" y="120.65" size="1.778" layer="95"/>
+<pinref part="JP6" gate="G$1" pin="1"/>
 </segment>
 </net>
@@
 <wire x1="158.75" y1="115.57" x2="137.16" y2="115.57" width="0.1524" layer="91"/>
 <label x="137.16" y="115.57" size="1.778" layer="95"/>
-</segment>
-</net>
+<pinref part="JP5" gate="G$1" pin="1"/>
+</segment>
+</net>

Commit message: labeling done
Parts:
- removed U5: MS621FE, Explore Labs EAGLE Library:MS621FE
- added C1: (no value), adafruit:SUPERCAP
Connections:
- net GND: now also C1.-; no longer U5.NEG
- net N$7: now also C1.+; no longer U5.POS
Changed lines of the file:
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@@
 <part name="U4" library="filters" deviceset="EPCOS-B9444" device=""/>
 <part name="U$27" library="microbuilder" deviceset="GND" device=""/>
-<part name="U5" library="Explore Labs EAGLE Library" deviceset="MS621FE" device=""/>
 <part name="U$28" library="microbuilder" deviceset="GND" device=""/>
 <part name="JP3" library="SparkFun-Connectors" deviceset="M01" device="NOSILK-KIT"/>
@@
 <part name="JP6" library="SparkFun-Connectors" deviceset="M01" device="NOSILK-KIT"/>
 <part name="JP7" library="SparkFun-Connectors" deviceset="M01" device="NOSILK-KIT"/>
+<part name="C1" library="adafruit" deviceset="SUPERCAP" device=""/>
 </parts>
 <sheets>
@@
 </instance>
 <instance part="U$27" gate="G$1" x="31.75" y="139.7"/>
-<instance part="U5" gate="G$1" x="236.22" y="158.75" rot="R90"/>
 <instance part="U$28" gate="G$1" x="8.89" y="153.67"/>
 <instance part="JP3" gate="G$1" x="224.79" y="115.57" rot="R180"/>
@@
 <instance part="JP6" gate="G$1" x="129.54" y="120.65"/>
 <instance part="JP7" gate="G$1" x="129.54" y="123.19"/>
+<instance part="C1" gate="G$1" x="238.76" y="158.75" rot="R90"/>
 </instances>
 <busses>
@@
 <pinref part="U$14" gate="G$1" pin="GND"/>
 <wire x1="243.84" y1="158.75" x2="243.84" y2="154.94" width="0.1524" layer="91"/>
-<pinref part="U5" gate="G$1" pin="NEG"/>
+<pinref part="C1" gate="G$1" pin="-"/>
 </segment>
 <segment>
@@
 <pinref part="SJ1" gate="G$1" pin="3"/>
 <wire x1="228.6" y1="156.21" x2="228.6" y2="158.75" width="0.1524" layer="91"/>
-<wire x1="228.6" y1="158.75" x2="231.14" y2="158.75" width="0.1524" layer="91"/>
+<wire x1="228.6" y1="158.75" x2="236.22" y2="158.75" width="0.1524" layer="91"/>
 <pinref part="R5" gate="G$1" pin="1"/>
 <wire x1="228.6" y1="158.75" x2="226.06" y2="158.75" width="0.1524" layer="91"/>
 <junction x="228.6" y="158.75"/>
-<pinref part="U5" gate="G$1" pin="POS"/>
-</segment>
-</net>
+<pinref part="C1" gate="G$1" pin="+"/>
+</segment>
+</net>
