File: electron-shields/asset-tracker/eagle/asset-tracker-v005/asset-tracker-v005.sch (EAGLE design)
At the start: 38 parts, among them J1 1X2-3.5MM, Q1 MPSA42, T1 DMG3415, U1 MAX-M8, U2 MAX2674, U3 LIS3DHTR, U4 EPCOS-B9444, X1 ELECTRON, X2 IPEX-20279-001E

Commit message: new gerbers made
Parts:
- JP3, JP4, JP5, JP6, JP7: device SparkFun-Connectors:M01NOSILK-KIT -> SparkFun-Connectors:M01SMD-4.5X1.5
Connections:
- net 3.3V: no longer R1.2
- net GND: now also U$26.-; no longer U$26.+, U$26.+1
- net GPS_VCC: now also R1.2
- net N$11: now also U$26.+; no longer U$26.-
Other:
- moved on the sheet: SJ1, U$26
Changed lines of the file:
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@@
 <layers>
 <layer number="1" name="Top" color="4" fill="1" visible="no" active="no"/>
-<layer number="2" name="Route2" color="1" fill="3" visible="no" active="no"/>
+<layer number="2" name="Route2" color="5" fill="1" visible="no" active="no"/>
 <layer number="3" name="Route3" color="4" fill="3" visible="no" active="no"/>
 <layer number="4" name="Route4" color="1" fill="4" visible="no" active="no"/>
@@
 <layer number="13" name="Route13" color="4" fill="5" visible="no" active="no"/>
 <layer number="14" name="Route14" color="1" fill="6" visible="no" active="no"/>
-<layer number="15" name="Route15" color="4" fill="6" visible="no" active="no"/>
+<layer number="15" name="Route15" color="11" fill="1" visible="no" active="no"/>
 <layer number="16" name="Bottom" color="1" fill="1" visible="no" active="no"/>
-<layer number="17" name="Pads" color="2" fill="1" visible="no" active="no"/>
-<layer number="18" name="Vias" color="2" fill="1" visible="no" active="no"/>
+<layer number="17" name="Pads" color="14" fill="1" visible="no" active="no"/>
+<layer number="18" name="Vias" color="14" fill="1" visible="no" active="no"/>
 <layer number="19" name="Unrouted" color="6" fill="1" visible="no" active="no"/>
 <layer number="20" name="Dimension" color="15" fill="1" visible="no" active="no"/>
-<layer number="21" name="tPlace" color="7" fill="1" visible="no" active="no"/>
+<layer number="21" name="tPlace" color="16" fill="1" visible="no" active="no"/>
 <layer number="22" name="bPlace" color="7" fill="1" visible="no" active="no"/>
 <layer number="23" name="tOrigins" color="15" fill="1" visible="no" active="no"/>
@@
 <layer number="27" name="tValues" color="7" fill="1" visible="no" active="no"/>
 <layer number="28" name="bValues" color="7" fill="1" visible="no" active="no"/>
-<layer number="29" name="tStop" color="7" fill="3" visible="no" active="no"/>
+<layer number="29" name="tStop" color="32" fill="3" visible="no" active="no"/>
 <layer number="30" name="bStop" color="7" fill="6" visible="no" active="no"/>
 <layer number="31" name="tCream" color="7" fill="4" visible="no" active="no"/>
@@
 <layer number="49" name="Reference" color="17" fill="6" visible="no" active="no"/>
 <layer number="50" name="dxf" color="7" fill="1" visible="no" active="no"/>
-<layer number="51" name="tDocu" color="14" fill="1" visible="no" active="no"/>
+<layer number="51" name="tDocu" color="24" fill="1" visible="no" active="no"/>
 <layer number="52" name="bDocu" color="7" fill="1" visible="no" active="no"/>
 <layer number="53" name="tGND_GNDA" color="7" fill="9" visible="no" active="no"/>
@@
 <part name="U$27" library="microbuilder" deviceset="GND" device=""/>
 <part name="U$28" library="microbuilder" deviceset="GND" device=""/>
-<part name="JP3" library="SparkFun-Connectors" deviceset="M01" device="NOSILK-KIT"/>
-<part name="JP4" library="SparkFun-Connectors" deviceset="M01" device="NOSILK-KIT"/>
-<part name="JP5" library="SparkFun-Connectors" deviceset="M01" device="NOSILK-KIT"/>
-<part name="JP6" library="SparkFun-Connectors" deviceset="M01" device="NOSILK-KIT"/>
-<part name="JP7" library="SparkFun-Connectors" deviceset="M01" device="NOSILK-KIT"/>
+<part name="JP3" library="SparkFun-Connectors" deviceset="M01" device="SMD-4.5X1.5"/>
+<part name="JP4" library="SparkFun-Connectors" deviceset="M01" device="SMD-4.5X1.5"/>
+<part name="JP5" library="SparkFun-Connectors" deviceset="M01" device="SMD-4.5X1.5"/>
+<part name="JP6" library="SparkFun-Connectors" deviceset="M01" device="SMD-4.5X1.5"/>
+<part name="JP7" library="SparkFun-Connectors" deviceset="M01" device="SMD-4.5X1.5"/>
 <part name="C1" library="adafruit" deviceset="SUPERCAP" device=""/>
 <part name="Q1" library="SparkFun-DiscreteSemi" deviceset="TRANSISTOR_NPN" device="MPSA42" value="MPSA42"/>
 <part name="R2" library="rcl" deviceset="R-US_" device="R0402" value="1K"/>
-<part name="U$29" library="microbuilder" deviceset="3.3V" device=""/>
 <part name="L2" library="inductors" deviceset="BLM15H" device="" technology="D102SN1"/>
 <part name="L3" library="inductors" deviceset="BLM15H" device="" technology="D102SN1"/>
@@
 <wire x1="147.32" y1="95.25" x2="248.92" y2="95.25" width="0.1524" layer="94" style="longdash"/>
 <wire x1="74.93" y1="95.25" x2="74.93" y2="0" width="0.1524" layer="94" style="longdash"/>
-<text x="234.95" y="140.97" size="1.778" layer="97">(HOLDER)</text>
+<text x="240.03" y="133.35" size="1.778" layer="97" rot="R90">(HOLDER)</text>
 <wire x1="147.32" y1="35.56" x2="147.32" y2="95.25" width="0.1524" layer="94" style="longdash"/>
 </plain>
@@
 <instance part="U$18" gate="G$1" x="5.08" y="48.26" rot="R270"/>
 <instance part="U$19" gate="G$1" x="52.07" y="58.42"/>
-<instance part="SJ1" gate="G$1" x="228.6" y="151.13" smashed="yes" rot="MR180">
-<attribute name="NAME" x="231.14" y="152.019" size="1.778" layer="95" rot="MR180"/>
+<instance part="SJ1" gate="G$1" x="232.41" y="151.13" smashed="yes" rot="MR180">
+<attribute name="NAME" x="234.95" y="152.019" size="1.778" layer="95" rot="MR180"/>
 </instance>
-<instance part="U$20" gate="G$1" x="241.3" y="137.16"/>
+<instance part="U$20" gate="G$1" x="234.95" y="128.27"/>
 <instance part="C10" gate="G$1" x="67.31" y="165.1" rot="R90"/>
 <instance part="U$21" gate="G$1" x="63.5" y="162.56"/>
@@
 <instance part="U$25" gate="G$1" x="201.93" y="74.93"/>
 <instance part="A1" gate="ANT" x="13.97" y="160.02"/>
-<instance part="U$26" gate="G$1" x="233.68" y="143.51"/>
+<instance part="U$26" gate="G$1" x="234.95" y="138.43" rot="R90"/>
 <instance part="R3" gate="G$1" x="182.88" y="167.64" rot="R90"/>
 <instance part="JP2" gate="G$1" x="220.98" y="62.23" rot="MR0"/>
@@
 <instance part="Q1" gate="G$1" x="105.41" y="125.73" rot="MR0"/>
 <instance part="R2" gate="G$1" x="115.57" y="125.73" rot="R180"/>
-<instance part="U$29" gate="G$1" x="82.55" y="138.43"/>
 <instance part="L2" gate="G$1" x="209.55" y="130.81" smashed="yes">
 <attribute name="NAME" x="204.47" y="132.1816" size="1.778" layer="95"/>
@@
 </segment>
 <segment>
-<pinref part="U$20" gate="G$1" pin="GND"/>
-<wire x1="241.3" y1="139.7" x2="241.3" y2="140.97" width="0.1524" layer="91"/>
-<pinref part="U$26" gate="G$1" pin="+"/>
-<wire x1="241.3" y1="140.97" x2="238.76" y2="140.97" width="0.1524" layer="91"/>
-<wire x1="238.76" y1="146.05" x2="241.3" y2="146.05" width="0.1524" layer="91"/>
-<wire x1="241.3" y1="146.05" x2="241.3" y2="140.97" width="0.1524" layer="91"/>
-<junction x="241.3" y="140.97"/>
-<pinref part="U$26" gate="G$1" pin="+1"/>
-</segment>
-<segment>
 <pinref part="C10" gate="G$1" pin="1"/>
 <pinref part="U$21" gate="G$1" pin="GND"/>
@@
 <pinref part="U$9" gate="G$1" pin="GND"/>
 <wire x1="102.87" y1="118.11" x2="102.87" y2="120.65" width="0.1524" layer="91"/>
+</segment>
+<segment>
+<pinref part="U$26" gate="G$1" pin="-"/>
+<pinref part="U$20" gate="G$1" pin="GND"/>
+<wire x1="234.95" y1="133.35" x2="234.95" y2="130.81" width="0.1524" layer="91"/>
 </segment>
 </net>
@@
 <pinref part="D3" gate="G$1" pin="A"/>
 <wire x1="208.28" y1="175.26" x2="208.28" y2="158.75" width="0.1524" layer="91"/>
-</segment>
-<segment>
-<pinref part="R1" gate="G$1" pin="2"/>
-<pinref part="U$29" gate="G$1" pin="3.3V"/>
-<wire x1="82.55" y1="135.89" x2="82.55" y2="133.35" width="0.1524" layer="91"/>
 </segment>
 </net>
@@
 <pinref part="U1" gate="MAX-M8" pin="V_BCKP"/>
 <wire x1="180.34" y1="143.51" x2="180.34" y2="151.13" width="0.1524" layer="91"/>
-<wire x1="180.34" y1="151.13" x2="223.52" y2="151.13" width="0.1524" layer="91"/>
+<wire x1="180.34" y1="151.13" x2="227.33" y2="151.13" width="0.1524" layer="91"/>
 <label x="186.69" y="151.13" size="1.778" layer="95"/>
 <pinref part="SJ1" gate="G$1" pin="2"/>
@@
 <label x="163.83" y="148.59" size="1.778" layer="95"/>
 </segment>
+<segment>
+<pinref part="R1" gate="G$1" pin="2"/>
+<wire x1="82.55" y1="133.35" x2="67.31" y2="133.35" width="0.1524" layer="91"/>
+<label x="68.58" y="133.35" size="1.778" layer="95"/>
+</segment>
 </net>
 <net name="N$2" class="0">
@@
 <segment>
 <pinref part="SJ1" gate="G$1" pin="3"/>
-<wire x1="228.6" y1="156.21" x2="228.6" y2="158.75" width="0.1524" layer="91"/>
-<wire x1="228.6" y1="158.75" x2="236.22" y2="158.75" width="0.1524" layer="91"/>
+<wire x1="232.41" y1="156.21" x2="232.41" y2="158.75" width="0.1524" layer="91"/>
+<wire x1="232.41" y1="158.75" x2="236.22" y2="158.75" width="0.1524" layer="91"/>
 <pinref part="R5" gate="G$1" pin="1"/>
-<wire x1="228.6" y1="158.75" x2="226.06" y2="158.75" width="0.1524" layer="91"/>
-<junction x="228.6" y="158.75"/>
+<wire x1="232.41" y1="158.75" x2="226.06" y2="158.75" width="0.1524" layer="91"/>
+<junction x="232.41" y="158.75"/>
 <pinref part="C1" gate="G$1" pin="+"/>
-</segment>
-</net>
-<net name="N$11" class="0">
-<segment>
-<pinref part="SJ1" gate="G$1" pin="1"/>
-<wire x1="228.6" y1="143.51" x2="228.6" y2="146.05" width="0.1524" layer="91"/>
-<pinref part="U$26" gate="G$1" pin="-"/>
 </segment>
 </net>
@@
 </segment>
 </net>
+<net name="N$11" class="0">
+<segment>
+<pinref part="SJ1" gate="G$1" pin="1"/>
+<pinref part="U$26" gate="G$1" pin="+"/>
+<wire x1="232.41" y1="143.51" x2="232.41" y2="146.05" width="0.1524" layer="91"/>
+</segment>
+</net>
