File: electron-shields/asset-tracker/eagle/asset-tracker-v006/asset-tracker-v006.sch (EAGLE design)
At the start: 45 parts, among them J1 1X2-3.5MM, Q1 MPSA42, T1 DMG3415, U1 MAX-M8, U3 LIS3DHTR, U4 RF_SWITCHSC-70-6, U6 BGA725L6-ALT, X1 ELECTRON, X2 IPEX-20279-001E

Commit message: v006 asset tracker gerber generated
Parts:
- removed C12: 10pF, rcl:C-EUC0402
- C6, C7, C8: device rcl:C-EUC0402 -> rcl:C-EUC0201
- U5: value (none) -> SAFFB1G56KB0F0A
Connections:
- net N$1 renamed LNA_OUT
- net N$12 renamed RF1
- net N$2 renamed ANT
- net N$3 renamed LNA_IN
- net N$4 renamed RF_SWITCH_OUT
- net N$42 renamed RF2
- net N$43 renamed EXT_ANT
- net N$5 renamed SAW_OUT
- net N$6 renamed TIMEPULSE
- net GND: no longer C12.1
- net GPS_VCC: no longer C12.2
Other:
- note added: "ACCELEROMETER"
- note added: "CONNECTORS"
- note added: "ELECTRON HEADER"
- note added: "GPS"
- note added: "LNA"
- note added: "RF SWITCH"
- note added: "SAW"
- moved on the sheet: C1, C11, C4, C9, D2, D3, JP3, JP4, L2, L3, Q1, R1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
